File: Electronics/arcreactor.kicad_pcb (KiCad board)
At the start: 2 copper layers, 127 x 127 mm, 36 parts, among them J1 Conn_01x01_Socket, J10 Conn_01x01_Socket, J11 ESP C3 mini, J12 Boost, J13 TP4056, J14 touch, J2 Conn_01x01_Socket, J3 Conn_01x01_Socket, J4 Conn_01x01_Socket, J5 Conn_01x01_Socket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

Commit message: pcb
Parts:
- J1, J10, J2, J3, J4, J5, J6, J7, J8, J9: footprint TestPoint:TestPoint_Pad_D2.0mm -> Library:SolderWirePad_1x01_SMD_2x5mm; moved to F.Cu
- R13: value R -> 33k
- R14: value R -> 10k
- moved J14 118.0 mm to (163.1, 104.1), turned to 180 degrees
- moved R15 84.2 mm to (123.7, 109.2)
- moved J7 79.1 mm to (117.1, 82.8)
- moved J2 76.7 mm to (98.6, 79.8)
- moved J12 74.6 mm to (123.2, 65.3), turned to 90 degrees
- moved Q7 74.4 mm to (123.6, 105.0), turned to 90 degrees
- moved R16 74.2 mm to (123.5, 99.8), turned to -90 degrees
- moved R9 72.9 mm to (118.6, 104.1)
- moved R7 72.4 mm to (113.6, 101.6)
- moved J5 70.9 mm to (112.3, 80.3)
- moved Q5 70.0 mm to (118.6, 99.9), turned to 90 degrees
- moved Q4 67.2 mm to (113.5, 97.4), turned to 90 degrees
- moved J10 66.8 mm to (118.5, 89.9)
- moved Q3 64.7 mm to (108.4, 94.8), turned to 90 degrees
- moved R10 64.0 mm to (118.5, 94.8), turned to -90 degrees
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Connections:
- J11 pad 9: GND -> boost out GND
- Q1 pad 2: GND -> boost out GND
- Q2 pad 2: GND -> boost out GND
- Q3 pad 2: GND -> boost out GND
- Q4 pad 2: GND -> boost out GND
- Q5 pad 2: GND -> boost out GND
- Q6 pad 3: GND -> boost out GND
- Q7 pad 2: GND -> boost out GND
- R1 pad 2: GND -> boost out GND
- R15 pad 2: GND -> boost out GND
- R3 pad 2: GND -> boost out GND
- R5 pad 2: GND -> boost out GND
- R7 pad 2: GND -> boost out GND
- R9 pad 2: GND -> boost out GND
Routing:
- net boost out +5V: track 0.00 -> 138.6 mm, vias 0 -> 1
- net LiPo +: track 0.00 -> 121.0 mm
- net LiPo -: track 0.00 -> 117.4 mm
- net Net-(J11-Pin_7): track 0.00 -> 63.8 mm
- net LED0: track 0.00 -> 34.0 mm
- net LED5: track 0.00 -> 29.0 mm
- net LED4: track 0.00 -> 23.9 mm
- net LED3: track 0.00 -> 18.8 mm
- net LED2: track 0.00 -> 13.4 mm
- net LED1: track 0.00 -> 8.71 mm
- net Net-(J14-Pin_2): track 0.00 -> 4.08 mm
- net Net-(J8-Pin_1): track 0.00 -> 3.84 mm
- net Net-(J6-Pin_1): track 0.00 -> 3.84 mm
- net Net-(J4-Pin_1): track 0.00 -> 3.84 mm
- net Net-(J10-Pin_1): track 0.00 -> 3.84 mm
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- added copper zone on F.Cu, net boost out GND
