File: Electronics/arcreactor.kicad_sch (KiCad schematic)
At the start: 21 parts, among them Q1 Q_NMOS_GSD, Q2 Q_NMOS_GSD, Q3 Q_NMOS_GSD, Q4 Q_NMOS_GSD, Q5 Q_NMOS_GSD, U1 WEMOS_C3_mini

Commit message: electronic
Parts:
- removed U1: WEMOS_C3_mini, RF_Module:WEMOS_C3_mini, symbol RF_Module:WEMOS_C3_mini
- added D0: LED, LED_SMD:LED_PLCC_2835_Handsoldering, symbol Device:LED
- added J1, J10, J2, J3, J4, J5, J6, J7, J8, J9: Conn_01x01_Socket, TestPoint:TestPoint_Pad_D2.0mm, symbol Connector:Conn_01x01_Socket
- added J11: ESP C3 mini, Connector_PinHeader_2.54mm:PinHeader_1x09_P2.54mm_Vertical, symbol Connector:Conn_01x09_Socket
- added J12: Boost, Connector_PinHeader_2.54mm:PinHeader_1x04_P2.54mm_Vertical, symbol Connector:Conn_01x04_Socket
- added J13: TP4056, Connector_PinHeader_2.54mm:PinHeader_1x04_P2.54mm_Vertical, symbol Connector:Conn_01x04_Socket
- added J14: touch, Connector_PinHeader_2.54mm:PinHeader_1x03_P2.54mm_Vertical, symbol Connector:Conn_01x03_Socket
- added Q6, Q7: Q_NMOS_GSD, Package_TO_SOT_SMD:SOT-23, symbol Transistor_FET:Q_NMOS_GSD
- added R13, R14, R16: R, Resistor_SMD:R_0805_2012Metric_Pad1.20x1.40mm_HandSolder, symbol Device:R
- added R15: 10k, Resistor_SMD:R_0805_2012Metric_Pad1.20x1.40mm_HandSolder, symbol Device:R
- R1, R3, R5, R7, R9: value R -> 10k; footprint (none) -> Resistor_SMD:R_0805_2012Metric_Pad1.20x1.40mm_HandSolder
- R10, R2, R4, R6, R8: value R -> 47; footprint (none) -> Resistor_SMD:R_0805_2012Metric_Pad1.20x1.40mm_HandSolder
Connections:
- net +5V: now also J13.1 (Pin_1); no longer D1.2 (A), D2.2 (A), D3.2 (A), D4.2 (A), D5.2 (A)
- net GND: now also R1.2, J11.9 (Pin_9), J13.2 (Pin_2), Q6.3 (D), Q7.2 (S), R15.2; no longer R2.2
- net LED0: now also J11.8 (Pin_8), Q7.1 (G), R15.1
- net LED1: now also R1.1, J11.2 (Pin_2); no longer R2.1
- net LED2: now also J11.3 (Pin_3)
- net LED3: now also J11.4 (Pin_4)
- net LED4: now also J11.5 (Pin_5)
- net LED5: now also J11.6 (Pin_6)
- net at Q1.3 (D): now also R2.2; no longer R1.2
- net at D2.1 (K), R4.1: now also J4.1 (Pin_1)
- net at D3.1 (K), R6.1: now also J6.1 (Pin_1)
- net at D4.1 (K), R8.1: now also J8.1 (Pin_1)
- net at D1.1 (K): now also R2.1, J2.1 (Pin_1); no longer R1.1
- net at D5.1 (K), R10.1: now also J10.1 (Pin_1)
- new net: J11.7 (Pin_7), R13.2, R14.1
- new net: Q7.3 (D), R16.2
- new net: D0.1 (K), R16.1
- new net: J14.2 (Pin_2), Q6.1 (G)
- new net LiPo +: J12.1 (Pin_1), J13.3 (Pin_3), J14.1 (Pin_1), R13.1
- new net LiPo -: J12.2 (Pin_2), J13.4 (Pin_4), J14.3 (Pin_3), Q6.2 (S), R14.2
- new net boost out +5V: D0.2 (A), D1.2 (A), D2.2 (A), D3.2 (A), D4.2 (A), D5.2 (A), J1.1 (Pin_1), J11.1 (Pin_1), J12.3 (Pin_3), J3.1 (Pin_1), J5.1 (Pin_1), J7.1 (Pin_1), J9.1 (Pin_1)
- new net boost out GND: J12.4 (Pin_4)
Other:
- moved on the sheet: R1, R2

Commit message: pcb
Parts:
- J1, J10, J2, J3, J4, J5, J6, J7, J8, J9: footprint TestPoint:TestPoint_Pad_D2.0mm -> Library:SolderWirePad_1x01_SMD_2x5mm
- R13: value R -> 33k
- R14: value R -> 10k
Connections:
- net GND: no longer J11.9 (Pin_9), Q1.2 (S), Q2.2 (S), Q3.2 (S), Q4.2 (S), Q5.2 (S), Q6.3 (D), Q7.2 (S), R1.2, R15.2, R3.2, R5.2, R7.2, R9.2
- net boost out GND: now also J11.9 (Pin_9), Q1.2 (S), Q2.2 (S), Q3.2 (S), Q4.2 (S), Q5.2 (S), Q6.3 (D), Q7.2 (S), R1.2, R15.2, R3.2, R5.2, R7.2, R9.2
